File: test.sch (KiCad schematic (older format))
At the start: 36 parts, among them J1 Serial header, J2 AVR-ISP-6, J3 5v Power, J4 INT0/1, J5 Servo, J6 Servo power, J7 I2C Header, Q1 2N7000, SW1 INT0, SW2 INT1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

Commit message: Schema error in PD5 fixed, sent to JLCPCB
Connections:
- net at J2.5 (~RST), Q1.2 (G), U1.1 (~RESET~/PC6): no longer U1.11 (PD5)
- no-connect marks 6 -> 8
Changed lines of the file:
@@
 $EndComp
-Wire Wire Line
-	2150 3300 1950 3300
 Wire Wire Line
 	2250 1450 2250 2300
@@
 	1    0    0    -1
 $EndComp
-Wire Wire Line
-	1950 3300 1950 4000
-Wire Wire Line
-	1950 4000 1750 4000
 NoConn ~ 1750 4200
 NoConn ~ 1750 3900
@@
 Text Label 1650 5250 0    50   ~ 0
 RXD
-Connection ~ 1950 3300
-Wire Wire Line
-	1950 3300 1750 3300
 $Comp
 L Transistor_FET:2N7000 Q1
@@
 	1900 6500 1550 6500
 Connection ~ 1550 6500
+Wire Wire Line
+	1750 3300 2150 3300
+NoConn ~ 1750 4000
+NoConn ~ 1750 4100
 $EndSCHEMATC
