File: test.kicad_pcb (KiCad board)
At the start: 2 copper layers, 80.3 x 41.7 mm, 36 parts, among them J1 Serial header, J2 AVR-ISP-6, J3 5v Power, J4 INT0/1, J5 Servo, J6 Servo power, J7 I2C Header, Q1 2N7000, SW1 INT0, SW2 INT1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

Commit message: Created new Gerbers
Other:
- board text added: "ATmega328P Development board rev1.1 (c) 2021 Jeroen Venema"
- board text removed: "ATmega328P Development board (c) 2021 Jeroen Venema"
